File: piprobe.kicad_pcb (KiCad board)
At the start: 4 copper layers, 15 x 34.1 mm, 28 parts, among them J1 USB_C_Receptacle_USB2.0, J2 Conn_01x03_Male, J3 Conn_01x06_Male, J4 Conn_01x10_Male, J5 Conn_01x10_Male, J6 Conn_01x06_Male, U1 TPS63020, U2 RP2040, U3 W25Q32JVZP, Y1 Crystal_GND24_Small

Commit message: ldo
Parts:
- removed C5: 100nF, Capacitor_SMD:C_0402_1005Metric_Pad0.74x0.62mm_HandSolder
- removed L1: 1.5uH, Inductor_SMD:L_0805_2012Metric
- removed R1: 180k, Resistor_SMD:R_0402_1005Metric_Pad0.72x0.64mm_HandSolder
- removed R2: 1M, Resistor_SMD:R_0402_1005Metric_Pad0.72x0.64mm_HandSolder
- C3: value 100uF -> 22uf; footprint Capacitor_SMD:C_1206_3216Metric -> Capacitor_SMD:C_0603_1608Metric
- C4: value 100uF -> 100uf
- U1: value TPS63020 -> MIC5524-3.3YMT-T5; footprint lib:QFN14-3X4MM -> lib:VREG_MIC5524-3.3YMT-T5
- moved C4 2.23 mm to (22.9, 27.2), turned to 180 degrees
- moved U1 1.05 mm to (22.9, 24.7), turned to 0 degrees
Connections:
- C4 pad 1: +3V3 -> GND
- C4 pad 2: GND -> +3V3
- U1 pad 1: Net-(C5-Pad1) -> +3V3
- U1 pad 3: Net-(R1-Pad1) -> +5V
- U1 pad 4: +3V3 -> +5V
Routing:
- net Net-(C5-Pad1): track 9.37 -> 0.00 mm, vias 2 -> 0
- net Net-(R1-Pad1): track 4.76 -> 0.00 mm
- net Net-(L1-Pad1): track 2.55 -> 0.00 mm
- net Net-(L1-Pad2): track 2.51 -> 0.00 mm
- net GND: track 106.4 -> 104.8 mm, vias 24 -> 26
- net +3V3: track 81.3 -> 82.4 mm, vias 13 -> 14
- removed copper zone on F.Cu, net Net-(C5-Pad1)
- removed copper zone on In1.Cu, net Net-(C5-Pad1)
Other:
- board text added: "500mA"
- board text added: "RS3236"
- board text added: "RS3236 中心焊盘为散热焊盘 非盘中孔 不塞孔"
- board text removed: "TPS63020"
